File: hardware/io.sch (KiCad schematic (older format))
At the start: 7 parts

Commit message: Partial updates for hardware revision 2
Parts:
- removed J?: USER PORT B, symbol Connector_Generic:Conn_02x06_Odd_Even
- added U?: WD65C22S, Package_DIP:DIP-40_W25.4mm_Socket, symbol 65xx:W65C22SxP
- added U?: Osc_8pin, symbol osc:Osc_8pin
- J?: value USER PORT A -> USER PORT; symbol Connector_Generic:Conn_02x06_Odd_Even -> Connector_Generic:Conn_02x12_Odd_Even
Connections:
- net labels added: +3V3, CA1-2, CA2-2, CB1-2, CB2-2, GCLK, INTR4B, IO2SELB, PA0-2, PA1-2, PA2-2, PA3-2, PA4-2, PA5-2, PA6-2, PA7-2, PA8-2, PB0-2, PB1-2, PB2-2, PB3-2, PB4-2, PB5-2, PB6-2, PB7-2
- net labels removed: EXPIRQ, RESET
- wire segments 166 -> 208

Commit message: Combine VIA, SPI, and UART into a single io.sch sheet. The serial.sch sheet is now just the serial ports and the line drivers.
Add ports.sch sheet for remaining I/O ports.
Parts:
- removed J?: USER PORT, symbol Connector_Generic:Conn_02x12_Odd_Even
- removed J?: EXPANSION, symbol Connector_Generic:Conn_02x24_Odd_Even
- removed J?: SERIAL A, symbol Connector:DB9_Male
- removed J?: SERIAL B, symbol Connector:DB9_Male
- removed U?: SC28L92, Package_LCC:PLCC-44_THT-Socket, symbol SC28L92:SC28L92
- removed U?: WD65C22S, Package_DIP:DIP-40_W25.4mm_Socket, symbol 65xx:W65C22SxP
- removed U?: Osc_8pin, symbol osc:Osc_8pin
- added C? (x6): 0.1uf, symbol Device:C_Small
- added U?: SC28L92, Package_LCC:PLCC-44_THT-Socket, symbol SC28L92:SC28L92
- added U?: ASFL1-3.6864MHZ-EK-T, symbol osc:Osc_8pin
- added U?: SPI65B, Package_QFP:TQFP-44_10x10mm_P0.8mm, symbol custom_chips:SPI65B
Connections:
- net labels added: RESET, R~W, SERCLK, SPI65_TDI, SPI_INT0, SPI_INT1, SPI_INT2, SPI_INT3, SPI_MISO, SPI_MOSI, SPI_SCLK, SPI_SS0, SPI_SS1, SPI_SS2, SPI_SS3, TCK, TDO, TMS, ~INTR1, ~INTR2, ~INTR3, ~IO1SEL, ~IO2SEL, ~IO3SEL, ~RD, ~RESET, ~WR, ϕ2
- net labels removed: +5V, A10, A11, A12, A13, A14, A15, A16, A17, A18, A19, A20, A21, A22, A23, A4, A5, A6, A7, A8, A9, ABORT, BE, CA1-2, CA2-2, CB1-2, CB2-2, GCLK, INTR1B, INTR2B, INTR4B, IO1SELB, IO2SELB, IOSEL2B, NMI, PA0-2, PA1-2, PA2-2, PA3-2, PA4-2, PA5-2, PA6-2, PA7-2, PA8-2, PB0-2, PB1-2, PB2-2, PB3-2, PB4-2, PB5-2, PB6-2, PB7-2, PHI2, RD, RDY, RES, RESB, ROMPROT, RWB, SER_CLK, VDA, VPA, WR
- wire segments 208 -> 149
- no-connect marks 9 -> 7
Other:
- moved on the sheet: U?
