File: hardware/memory.sch (KiCad schematic (older format))
At the start: 3 parts

Commit message: Partial updates for hardware revision 2
Parts:
- removed U?: 28C256, symbol Memory_EEPROM:28C256
- added C? (x3): 0.1uf, symbol Device:C_Small
- added U?: SST39VF040-70-4I-NHE, Package_LCC:PLCC-32_11.4x14.0mm_P1.27mm, symbol cole-2-rescue:SST39VF040-Memory_Flash
Connections:
- net labels added: +3V3, ~RAM1CS, ~RAM2CS, ~RD, ~ROMCS, ~WR
- net labels removed: +5V, RAM1CSB, RAM2CSB, RDB, ROMCSB, ROMWRB, WRB
- wire segments 92 -> 108
Other:
- moved on the sheet: U?
